File: output.kicad_sch (KiCad schematic)
At the start: 35 parts, among them J3 AudioJack2_Ground_Switch, Q1 BSS138, U3 LM358B, U7 MCP4725xxx-xCH

Commit message: Changed ESD diodes and adjusted some parts
Parts:
- C22, C23: value 100nF -> 0.1uF
- D12, D13: LCSC C52148407 -> C169433
Changed lines of the file:
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@@
 			)
 		)
-		(property "LCSC" "C52148407"
+		(property "LCSC" "C169433"
 			(at 190.5 41.91 0)
 			(effects
@@
 			)
 		)
-		(property "LCSC" "C52148407"
+		(property "LCSC" "C169433"
 			(at 124.46 151.13 90)
 			(effects
@@
 			)
 		)
-		(property "Value" "100nF"
+		(property "Value" "0.1uF"
 			(at 180.34 105.41 0)
 			(effects
@@
 			)
 		)
-		(property "Value" "100nF"
+		(property "Value" "0.1uF"
 			(at 135.89 105.41 0)
 			(effects
