File: mcu.kicad_sch (KiCad schematic)
At the start: 47 parts, among them J1 USB_C_Receptacle_USB2.0_16P, J4 Conn_01x03_Pin, J5 Conn_01x03_Pin, J6 Conn_02x04_Odd_Even, J7 AudioJack2_Ground_Switch, SW4 RotaryEncoder_Switch, SW5 RESET, SW6 BOOTSEL, U1 RP2040, U5 W25Q64JVSSIQ, U6 ADS1015IDGS, Y1 XYDBPCNANF-12MHZ

Commit message: Changed ESD diodes and adjusted some parts
Parts:
- C24, C3: value 100nF -> 0.1uF
- D10, D11, D9: footprint Diode_SMD:D_0201_0603Metric -> Diode_SMD:D_0402_1005Metric; LCSC C52994072 -> C316049
- J6: now not fitted; now left out of the parts list
Changed lines of the file:
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@@
 			)
 		)
-		(property "Footprint" "Diode_SMD:D_0201_0603Metric"
+		(property "Footprint" "Diode_SMD:D_0402_1005Metric"
 			(at 222.25 140.97 0)
 			(effects
@@
 			)
 		)
-		(property "LCSC" "C52994072"
+		(property "LCSC" "C316049"
 			(at 222.25 135.89 0)
 			(effects
@@
 			)
 		)
-		(property "Footprint" "Diode_SMD:D_0201_0603Metric"
+		(property "Footprint" "Diode_SMD:D_0402_1005Metric"
 			(at 222.25 120.65 0)
 			(effects
@@
 			)
 		)
-		(property "LCSC" "C52994072"
+		(property "LCSC" "C316049"
 			(at 222.25 115.57 0)
 			(effects
@@
 			)
 		)
-		(property "Value" "100nF"
+		(property "Value" "0.1uF"
 			(at 247.65 123.19 0)
 			(effects
@@
 			)
 		)
-		(property "Footprint" "Diode_SMD:D_0201_0603Metric"
+		(property "Footprint" "Diode_SMD:D_0402_1005Metric"
 			(at 222.25 135.89 0)
 			(effects
@@
 			)
 		)
-		(property "LCSC" "C52994072"
+		(property "LCSC" "C316049"
 			(at 222.25 130.81 0)
 			(effects
@@
 			)
 		)
-		(property "Value" "100nF"
+		(property "Value" "0.1uF"
 			(at 252.73 148.59 0)
 			(effects
@@
 		(unit 1)
 		(exclude_from_sim no)
-		(in_bom yes)
+		(in_bom no)
 		(on_board yes)
-		(dnp no)
+		(dnp yes)
 		(fields_autoplaced yes)
 		(property "Reference" "J6"

Commit message: Updated D14 to 0402
Parts:
- D14: footprint Diode_SMD:D_0201_0603Metric -> Diode_SMD:D_0402_1005Metric; LCSC C52994072 -> C316049
Changed lines of the file:
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@@
 			)
 		)
-		(property "Footprint" "Diode_SMD:D_0201_0603Metric"
+		(property "Footprint" "Diode_SMD:D_0402_1005Metric"
 			(at 160.02 69.85 0)
 			(effects
@@
 			)
 		)
-		(property "LCSC" "C52994072"
+		(property "LCSC" "C316049"
 			(at 165.1 69.85 0)
 			(effects
