File: mcu.kicad_sch (KiCad schematic)
At the start: 63 parts, among them J1 USB_C_Receptacle_USB2.0_16P, J2 Conn_01x04_Pin, J3 AudioJack2_Ground_Switch, J4 AudioJack2_Ground_Switch, J5 Conn_01x04_Pin, J6 Conn_01x04_Pin, J7 AudioJack2_Ground_Switch, Q2 BSS138, SW4 RotaryEncoder_Switch, SW7 BTN, SW8 BTN, SW9 BTN, U1 STM32G0B1RBTx, U8 LM358B

Commit message: Added charge indicator LED, upped charge pump capacitor bank voltage rating for more headroom
Parts:
- C29, C30, C42, C43, C44: footprint Capacitor_SMD:C_0603_1608Metric_Pad1.08x0.95mm_HandSolder -> Capacitor_SMD:C_0805_2012Metric; LCSC C19666 -> C1779
Changed lines of the file:
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@@
 			)
 		)
-		(property "Footprint" "Capacitor_SMD:C_0603_1608Metric_Pad1.08x0.95mm_HandSolder"
+		(property "Footprint" "Capacitor_SMD:C_0805_2012Metric"
 			(at 195.2752 71.12 0)
 			(hide yes)
@@
 			)
 		)
-		(property "LCSC" "C19666"
+		(property "LCSC" "C1779"
 			(at 194.31 67.31 0)
 			(hide yes)
@@
 			)
 		)
-		(property "Footprint" "Capacitor_SMD:C_0603_1608Metric_Pad1.08x0.95mm_HandSolder"
+		(property "Footprint" "Capacitor_SMD:C_0805_2012Metric"
 			(at 155.9052 71.12 0)
 			(hide yes)
@@
 			)
 		)
-		(property "LCSC" "C19666"
+		(property "LCSC" "C1779"
 			(at 154.94 67.31 0)
 			(hide yes)
@@
 			)
 		)
-		(property "Footprint" "Capacitor_SMD:C_0603_1608Metric_Pad1.08x0.95mm_HandSolder"
+		(property "Footprint" "Capacitor_SMD:C_0805_2012Metric"
 			(at 181.3052 71.12 0)
 			(hide yes)
@@
 			)
 		)
-		(property "LCSC" "C19666"
+		(property "LCSC" "C1779"
 			(at 180.34 67.31 0)
 			(hide yes)
@@
 			)
 		)
-		(property "Footprint" "Capacitor_SMD:C_0603_1608Metric_Pad1.08x0.95mm_HandSolder"
+		(property "Footprint" "Capacitor_SMD:C_0805_2012Metric"
 			(at 168.6052 71.12 0)
 			(hide yes)
@@
 			)
 		)
-		(property "LCSC" "C19666"
+		(property "LCSC" "C1779"
 			(at 167.64 67.31 0)
 			(hide yes)
@@
 			)
 		)
-		(property "Footprint" "Capacitor_SMD:C_0603_1608Metric_Pad1.08x0.95mm_HandSolder"
+		(property "Footprint" "Capacitor_SMD:C_0805_2012Metric"
 			(at 211.7852 71.12 0)
 			(hide yes)
@@
 			)
 		)
-		(property "LCSC" "C19666"
+		(property "LCSC" "C1779"
 			(at 210.82 67.31 0)
 			(hide yes)

Commit message: Some minor clean ups
Parts:
- renumbered C30 to C10, C37 to C11, C45 to C12, C42 to C13, C43 to C14, C46 to C15, C39 to C16, C44 to C17, C24 to C18, C3 to C19, C28 to C4, C50 to C5, C48 to C6, C49 to C7, C47 to C8, C29 to C9, D11 to D10, D10 to D11, D18 to D12, D19 to D13, D20 to D15, D21 to D5, D15 to D6, D16 to D7, D17 to D8, J5 to J1, J1 to J2, J7 to J3, J6 to J4, J2 to J5, J3 to J6, J4 to J7, Q2 to Q1, R51 to R10, R33 to R11, R40 to R12, R41 to R13, R9 to R14, R10 to R15, R44 to R16, R45 to R17, R37 to R18, R42 to R19, R47 to R20, R46 to R21, R49 to R22, R48 to R23, R34 to R3, R35 to R4, R50 to R5, R36 to R6, R38 to R7, R39 to R8, R43 to R9, SW8 to SW2, SW9 to SW3, SW7 to SW5, U8 to U3, U1 to U4
Connections:
- net BODY_ELECTRODE: now also J7.R, J7.S
- net FOLLICLE_ELECTRODE: now also J6.R, J6.S
- net GND: now also SW4.MP
- no-connect marks 9 -> 5

Commit message: Make buzzer single sided for simplicity
Connections:
- net GND: now also BZ1.2 (-)
- net BUZZER2: no longer names the net of U4.2 (PC12)
- net BUZZER2: no longer BZ1.2 (-)
Changed lines of the file:
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@@
 	(wire
 		(pts
-			(xy 27.94 162.56) (xy 43.18 162.56)
-		)
-		(stroke
-			(width 0)
-			(type default)
-		)
-	)
-	(wire
-		(pts
 			(xy 266.7 146.05) (xy 266.7 143.51)
 		)
@@
 		)
 	)
-	(label "BUZZER2"
-		(at 149.86 191.77 0)
-		(effects
-			(font
-				(size 1.27 1.27)
-			)
-			(justify left bottom)
-		)
-	)
 	(label "PA15"
 		(at 129.54 147.32 0)
@@
 		)
 	)
-	(label "BUZZER2"
-		(at 27.94 162.56 0)
-		(effects
-			(font
-				(size 1.27 1.27)
-			)
-			(justify left bottom)
-		)
-	)
 	(label "USB_SENSE"
 		(at 250.19 116.84 0)
@@
 					(unit 1)
 				)
+			)
+		)
+	)
+	(symbol
+		(lib_id "power:GND")
+		(at 149.86 191.77 0)
+		(unit 1)
+		(body_style 1)
+		(exclude_from_sim no)
+		(in_bom yes)
+		(on_board yes)
+		(in_pos_files yes)
+		(dnp no)
+		(property "Reference" "#PWR060"
+			(at 149.86 198.12 0)
+			(hide yes)
+			(show_name no)
+			(do_not_autoplace no)
+			(effects
+				(font
+					(size 1.27 1.27)
+				)
+			)
+		)
+		(property "Value" "GND"
+			(at 149.86 195.9031 0)
+			(show_name no)
+			(do_not_autoplace no)
+			(effects
+				(font
+					(size 1.27 1.27)
+				)
+			)
+		)
+		(property "Footprint" ""
+			(at 149.86 191.77 0)
+			(hide yes)
+			(show_name no)
+			(do_not_autoplace no)
+			(effects
+				(font
+					(size 1.27 1.27)
+				)
+			)
+		)
+		(property "Datasheet" ""
+			(at 149.86 191.77 0)
+			(hide yes)
+			(show_name no)
+			(do_not_autoplace no)
+			(effects
+				(font
+					(size 1.27 1.27)
+				)
+			)
+		)
+		(property "Description" "Power symbol creates a global label with name \"GND\" , ground"
+			(at 149.86 191.77 0)
+			(hide yes)
+			(show_name no)
+			(do_not_autoplace no)
+			(effects
+				(font
+					(size 1.27 1.27)
+				)
+			)
+		)
+		(pin "1"
+		)
+		(instances
+			(project "hair-electrolysis-machine"
+				(path "/724ce5ca-e5bf-4553-b755-84be7690a548/cdc4525c-ab23-4870-9f65-db2094403a54"
+					(reference "#PWR060")
+					(unit 1)
+				)
