File: mcu.kicad_sch (KiCad schematic)
At the start: 63 parts, among them J1 Conn_01x04_Pin, J2 USB_C_Receptacle_USB2.0_16P, J3 AudioJack2_Ground_Switch, J4 Conn_01x04_Pin, J5 Conn_01x04_Pin, J6 AudioJack2_Ground_Switch, J7 AudioJack2_Ground_Switch, Q1 BSS138, SW2 BTN, SW3 BTN, SW4 RotaryEncoder_Switch, SW5 BTN, U3 LM358B, U4 STM32G0B1RBTx

Commit message: change jack pinout and charge limiting
limit charge speed to be more conservative and change jack pins used so there's zero overlap between pedal and stylus
Connections:
- net FOLLICLE_ELECTRODE: no longer J6.R, J6.S
- net GND: no longer J3.R, J3.S
- net TRIGGER: now also J3.R; no longer J3.T
- net at J3.RN: now also J3.TN
- no-connect marks 2 -> 4
Other:
- note removed: "Current 0mA-2.426mA w/ 0.6uA stepping"
- moved on the sheet: R19

Commit message: v4.1, see commit for details
Added passthrough hole for battery wires for users soldering batteries in
Cleared ground plane under screw holes
Uses only 3.5mm tip for stylus and sleeve for the pedal
Better anchoring for the 2.5mm jack for improved durability
Connections:
- net GND: now also J3.R, J3.T
- net TRIGGER: now also J3.S; no longer J3.R
- net at J3.RN: no longer J3.TN
Other:
- moved on the sheet: C4, R14, R15, SW3
